File: smt/input-power-board-smt.kicad_pcb (KiCad board)
At the start: 2 copper layers, 38.6 x 29 mm, 11 parts, among them J2 HEADER, J2A1 SCREW, J3 HEADER, J3A1 SCREW, J4 HEADER, J4A1 SCREW, J5 BARREL_JACK, U1 NCP1117-5V, U2 NCP1117-3.3V

Commit message: Added outline to assembly drawing.
Other:
- board text added: "8/23/16"
- board text added: "Input Power Board SMT v1.1"
Changed lines of the file:
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@@
 (kicad_pcb (version 4) (host pcbnew 4.0.1-3.201512221402+6198~38~ubuntu14.04.1-stable)
   (general
-    (links 25)
-    (no_connects 11)
-    (area 107.620999 83.236999 195.910202 129.870202)
+    (links 21)
+    (no_connects 0)
+    (area 107.595999 79.526 195.910202 129.870202)
     (thickness 1.6)
-    (drawings 17)
+    (drawings 23)
     (tracks 26)
     (zones 0)
@@
   )
   (setup
-    (last_trace_width 0.762)
+    (last_trace_width 0.1524)
     (user_trace_width 0.1524)
     (user_trace_width 0.254)
@@
     (visible_elements FFFEDF7D)
     (pcbplotparams
-      (layerselection 0x3d0fc_80000001)
+      (layerselection 0x20000_00000000)
       (usegerberextensions true)
       (excludeedgelayer true)
@@
       (net 1 GND))
   )
+  (gr_text 8/23/16 (at 140.97 114.3) (layer F.Fab)
+    (effects (font (size 1.5 1.5) (thickness 0.3)) (justify mirror))
+  )
+  (gr_text "Input Power Board SMT v1.1" (at 129.54 81.026) (layer F.Fab)
+    (effects (font (size 1.5 1.5) (thickness 0.3)))
+  )
+  (gr_line (start 107.696 83.312) (end 146.304 83.312) (layer F.Fab) (width 0.2))
+  (gr_line (start 107.696 112.268) (end 107.696 83.312) (layer F.Fab) (width 0.2))
+  (gr_line (start 146.304 112.268) (end 107.696 112.268) (layer F.Fab) (width 0.2))
+  (gr_line (start 146.304 83.312) (end 146.304 112.268) (layer F.Fab) (width 0.2))
   (gr_text NCP1117-5V (at 129.54 90.424 90) (layer F.SilkS)
     (effects (font (size 1.2 1.2) (thickness 0.2)))
@@
     (effects (font (size 1.2 1.2) (thickness 0.2)))
   )
-  (gr_text "VIN INPUT" (at 114.808 102.616 360) (layer F.SilkS)
+  (gr_text "VIN INPUT" (at 114.808 102.616) (layer F.SilkS)
     (effects (font (size 1.5 1.5) (thickness 0.3)))
   )
@@
     (effects (font (size 1.016 1.016) (thickness 0.2032)))
   )
-  (gr_text wickerbox.net (at 138.684 110.236 360) (layer B.SilkS)
+  (gr_text wickerbox.net (at 138.684 110.236) (layer B.SilkS)
     (effects (font (size 1.016 1.016) (thickness 0.2032)) (justify mirror))
   )
