File: th/input-power-board-th.kicad_pcb (KiCad board)
At the start: 2 copper layers, 41.7 x 25.9 mm, 13 parts, among them J1 HEADER, J1A1 SCREW, J2 HEADER, J2A1 SCREW, J3 HEADER, J3A1 SCREW, J4 HEADER, J4A1 SCREW

Commit message: Added outline to assembly drawing.
Other:
- board text added: "8/23/16"
- board text added: "Input Power Board TH v1.1"
Changed lines of the file:
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@@
     (links 25)
     (no_connects 0)
-    (area 97.358139 85.3988 195.910202 129.870202)
+    (area 97.358139 82.828 195.910202 129.870202)
     (thickness 1.6)
-    (drawings 18)
+    (drawings 24)
     (tracks 32)
     (zones 0)
@@
     (visible_elements FFFEDF7D)
     (pcbplotparams
-      (layerselection 0x3d0fc_80000001)
+      (layerselection 0x20000_00000000)
       (usegerberextensions true)
       (excludeedgelayer true)
@@
       (net 1 GND))
   )
+  (gr_text "Input Power Board TH v1.1" (at 123.952 84.328) (layer F.Fab)
+    (effects (font (size 1.5 1.5) (thickness 0.3)))
+  )
+  (gr_text 8/23/16 (at 133.858 114.046) (layer F.Fab)
+    (effects (font (size 1.5 1.5) (thickness 0.3)))
+  )
+  (gr_line (start 139.7 112.268) (end 139.7 86.36) (layer F.Fab) (width 0.2))
+  (gr_line (start 98.044 112.268) (end 139.7 112.268) (layer F.Fab) (width 0.2))
+  (gr_line (start 98.044 86.36) (end 98.044 112.268) (layer F.Fab) (width 0.2))
+  (gr_line (start 139.7 86.36) (end 98.044 86.36) (layer F.Fab) (width 0.2))
   (gr_text 3.3V (at 129.6924 102.7684 90) (layer F.SilkS)
     (effects (font (size 1.2 1.2) (thickness 0.2)))
